Commit message: Added X and O meshes, tested erasing in sim, bugfixes

File: src/end_effector/urdf/ur_with_pen_holder.xacro (robot description, xacro)
@@ -13,7 +13,4 @@
         <box size="0.1 0.1 0.1"/>  <!-- Length, Width, Height -->
       </geometry>
-      <material name="orange">
-        <color rgba="1.025 0.5 0.0 1.0"/>
-      </material>
     </visual>
     <collision>
