Commit message: Wk12 Monday testing

File: src/end_effector/urdf/ur_with_end_effector.xacro (robot description, xacro)
@@ -5,9 +5,10 @@
   <xacro:arg name="ur_type" default="ur5e"/>
   <xacro:include filename="$(find ur_description)/urdf/ur.urdf.xacro"/>
-  <!-- End-effector -->
+  <!-- End-effector with mesh -->
   <link name="end_effector_dual">
     <visual>
+      <origin xyz="-0.06 -0.065 0.085" rpy="3.141 0 1.5708"/>
       <geometry>
-        <mesh filename="package://end_effector/meshes/end_effector_dual.STL"/>
+        <mesh filename="package://end_effector/meshes/end_effector_dual.STL" scale="1 1 1"/>
       </geometry>
       <material name="gray">
@@ -16,10 +17,11 @@
     </visual>
     <collision>
+      <origin xyz="-0.06 -0.065 0.085" rpy="3.141 0 1.5708"/>
       <geometry>
-        <!-- Use simplified collision mesh or same mesh -->
-        <mesh filename="package://end_effector/meshes/end_effector_dual.STL"/>
+        <box size="0.01 0.01 0.01"/>
       </geometry>
     </collision>
     <inertial>
+      <origin xyz="0 0 0" rpy="0 0 0"/>
       <mass value="2.0"/>
       <inertia
@@ -29,9 +31,8 @@
     </inertial>
   </link>
-  <!-- Fixed joint attaching to tool0 -->
   <joint name="simple_ee_joint" type="fixed">
     <parent link="tool0"/>
     <child link="end_effector_dual"/>
-    <origin xyz="0 0 0" rpy="0 0 0"/>
+    <origin xyz="0.0 0.0 0.02" rpy="0 0 0"/>
   </joint>
 </robot>

Commit message: Adjusted end-effector parameters

File: src/end_effector/urdf/ur_with_end_effector.xacro (robot description, xacro)
@@ -19,14 +19,14 @@
       <origin xyz="-0.06 -0.065 0.085" rpy="3.141 0 1.5708"/>
       <geometry>
-        <box size="0.01 0.01 0.01"/>
+        <box size="0.1 0.1 0.1"/>
       </geometry>
     </collision>
     <inertial>
       <origin xyz="0 0 0" rpy="0 0 0"/>
-      <mass value="2.0"/>
+      <mass value="1.0"/>
       <inertia
-        ixx="0.01625" ixy="0.0" ixz="0.0"
-        iyy="0.0085" iyz="0.0"
-        izz="0.00425"/>
+        ixx="0.0016667" ixy="0.0" ixz="0.0"
+        iyy="0.0016667" iyz="0.0"
+        izz="0.0016667"/>
     </inertial>
   </link>
